Commit message: Update lidar.xacro
rotate lidar to match in rviz

File: description/lidar.xacro (robot description, xacro)
@@ -4,5 +4,5 @@
         <parent link="chassis"/>
         <child link="laser_frame"/>
-        <origin xyz="0.1 0 0.175" rpy="0 0 0"/>
+        <origin xyz="0.1 0 0.175" rpy="0 0 -1.5708"/>
     </joint>
     <link name="laser_frame">

Commit message: Update lidar.xacro
Updated lidar dimensions

File: description/lidar.xacro (robot description, xacro)
@@ -4,10 +4,10 @@
         <parent link="chassis"/>
         <child link="laser_frame"/>
-        <origin xyz="0.1 0 0.175" rpy="0 0 -1.5708"/>
+        <origin xyz="0.145 0 0.865" rpy="0 0 -1.5708"/>
     </joint>
     <link name="laser_frame">
         <visual>
             <geometry>
-                <cylinder radius="0.05" length="0.04"/>
+                <cylinder radius="0.0165" length="0.033"/>
             </geometry>
             <material name="red"/>
@@ -25,5 +25,5 @@
         <material>Gazebo/Red</material>
         <sensor name="laser" type="ray">
-            <pose> 0 0 0 0 0 0 </pose>
+            <pose> 0 0 0.0165 0 0 0 </pose>
             <visualize>false</visualize>
             <update_rate>10</update_rate>

Commit message: Update lidar.xacro
Fixed lidar height

File: description/lidar.xacro (robot description, xacro)
@@ -4,5 +4,5 @@
         <parent link="chassis"/>
         <child link="laser_frame"/>
-        <origin xyz="0.145 0 0.865" rpy="0 0 -1.5708"/>
+        <origin xyz="0.145 0 0.0865" rpy="0 0 -1.5708"/>
     </joint>
     <link name="laser_frame">

Commit message: Update lidar.xacro
Updated lidar position

File: description/lidar.xacro (robot description, xacro)
@@ -4,5 +4,5 @@
         <parent link="chassis"/>
         <child link="laser_frame"/>
-        <origin xyz="0.145 0 0.0865" rpy="0 0 -1.5708"/>
+        <origin xyz="0.65 0 0.0865" rpy="0 0 -1.5708"/>
     </joint>
     <link name="laser_frame">

Commit message: Revert "Update lidar.xacro"
This reverts commit 681c4cb666e582fd9d9c3a1cae43200b53eb4504.

File: description/lidar.xacro (robot description, xacro)
@@ -4,5 +4,5 @@
         <parent link="chassis"/>
         <child link="laser_frame"/>
-        <origin xyz="0.65 0 0.0865" rpy="0 0 -1.5708"/>
+        <origin xyz="0.145 0 0.0865" rpy="0 0 -1.5708"/>
     </joint>
     <link name="laser_frame">

Commit message: Update lidar.xacro
Updated lidar position

File: description/lidar.xacro (robot description, xacro)
@@ -4,5 +4,5 @@
         <parent link="chassis"/>
         <child link="laser_frame"/>
-        <origin xyz="0.145 0 0.0865" rpy="0 0 -1.5708"/>
+        <origin xyz="0.065 0 0.0865" rpy="0 0 -1.5708"/>
     </joint>
     <link name="laser_frame">
