Commit message: Update imu.xacro
set bno055 to z=0.0 wich is correct

File: description/imu.xacro (robot description, xacro)
@@ -3,5 +3,5 @@
     <xacro:property name="imu_parent_link" value="chassis" />
     <xacro:property name="imu_link_name" value="bno055" />
-    <xacro:property name="imu_pos_x" value="0.0" />  <xacro:property name="imu_pos_y" value="0.0" />  <xacro:property name="imu_pos_z" value="0.01" /> <joint name="imu_joint" type="fixed">
+    <xacro:property name="imu_pos_x" value="0.0" />  <xacro:property name="imu_pos_y" value="0.0" />  <xacro:property name="imu_pos_z" value="0.0" /> <joint name="imu_joint" type="fixed">
         <parent link="${imu_parent_link}"/>
         <child link="${imu_link_name}"/>

Commit message: Update imu.xacro

File: description/imu.xacro (robot description, xacro)
@@ -1,5 +1,5 @@
 <?xml version="1.0"?>
 <robot xmlns:xacro="http://www.ros.org/wiki/xacro" >
-    <xacro:property name="imu_parent_link" value="chassis" />
+    <xacro:property name="imu_parent_link" value="base_link" />
     <xacro:property name="imu_link_name" value="bno055" />
     <xacro:property name="imu_pos_x" value="0.0" />  <xacro:property name="imu_pos_y" value="0.0" />  <xacro:property name="imu_pos_z" value="0.0" /> <joint name="imu_joint" type="fixed">
