Commit message: Update robot_core.xacro
test in right_wheel

File: description/robot_core.xacro (robot description, xacro)
@@ -86,5 +86,5 @@
         <child link="right_wheel"/>
         <origin xyz="0 -0.175 0" rpy="${pi/2} 0 0"/>
-        <axis xyz="0 0 -1"/>
+        <axis xyz="0 0 1"/>
     </joint>
     <link name="right_wheel">

Commit message: Update robot_core.xacro
right_wheel back to 1 and higher mu for caster_wheel

File: description/robot_core.xacro (robot description, xacro)
@@ -86,5 +86,5 @@
         <child link="right_wheel"/>
         <origin xyz="0 -0.175 0" rpy="${pi/2} 0 0"/>
-        <axis xyz="0 0 1"/>
+        <axis xyz="0 0 -1"/>
     </joint>
     <link name="right_wheel">
@@ -131,6 +131,6 @@
     <gazebo reference="caster_wheel">
         <material>Gazebo/Black</material>
-        <mu1 value="0.001"/>
-        <mu2 value="0.001"/>
+        <mu1 value="0.1"/>
+        <mu2 value="0.1"/>
     </gazebo>
 </robot>

Commit message: Update robot_core.xacro
Fixed chassis

File: description/robot_core.xacro (robot description, xacro)
@@ -46,5 +46,5 @@
         <parent link="base_link"/>
         <child link="chassis"/>
-        <origin xyz="${-wheel_offset_x} 0 ${+wheel_offset_z}"/>
+        <origin xyz="${wheel_offset_x} 0 ${+wheel_offset_z}"/>
     </joint>
     <link name="chassis">

Commit message: Revert "Update robot_core.xacro"
This reverts commit 769c402e024dcbde7a6e43ce38dfe29034ed12ee.

File: description/robot_core.xacro (robot description, xacro)
@@ -46,5 +46,5 @@
         <parent link="base_link"/>
         <child link="chassis"/>
-        <origin xyz="${wheel_offset_x} 0 ${+wheel_offset_z}"/>
+        <origin xyz="${-wheel_offset_x} 0 ${+wheel_offset_z}"/>
     </joint>
     <link name="chassis">

Commit message: Update robot_core.xacro

File: description/robot_core.xacro (robot description, xacro)
@@ -46,5 +46,5 @@
         <parent link="base_link"/>
         <child link="chassis"/>
-        <origin xyz="${-wheel_offset_x} 0 ${+wheel_offset_z}"/>
+        <origin xyz="${-chassis_length + wheel_offset_x} 0 ${+wheel_offset_z}"/>
     </joint>
     <link name="chassis">

Commit message: Replace orange material with black in robot_core.xacro
The 'orange' material definition was removed and replaced with a 'black' material definition in the robot_core.xacro file. This may affect the appearance of components using this material.

File: description/robot_core.xacro (robot description, xacro)
@@ -19,6 +19,6 @@
         <color rgba="1 1 1 1" />
     </material>
-    <material name="orange">
-        <color rgba="1 0.3 0.1 1"/>
+    <material name="black">
+        <color rgba="0 0 0 1"/>
     </material>
     <material name="blue">

Commit message: Change chassis material from orange to black
Updated the chassis visual and Gazebo material from orange to black for consistency in appearance.

File: description/robot_core.xacro (robot description, xacro)
@@ -54,5 +54,5 @@
                 <box size="${chassis_length} ${chassis_width} ${chassis_height}"/>
             </geometry>
-            <material name="orange"/>
+            <material name="black"/>
         </visual>
         <collision>
@@ -67,5 +67,5 @@
     </link>
     <gazebo reference="chassis">
-        <material>Gazebo/Orange</material>
+        <material>Gazebo/Black</material>
     </gazebo>
     <!-- LEFT WHEEL LINK -->

Commit message: Fix caster wheel Z offset calculation in xacro
Corrects the formula for 'caster_wheel_offset_z' by negating 'wheel_offset_z', ensuring the caster wheel is positioned accurately in the robot model.

File: description/robot_core.xacro (robot description, xacro)
@@ -15,5 +15,5 @@
     <xacro:property name="caster_wheel_mass" value="0.01"/>
     <xacro:property name="caster_wheel_offset_x" value="0.03"/>
-    <xacro:property name="caster_wheel_offset_z" value="${wheel_offset_z - wheel_radius + caster_wheel_radius}"/>
+    <xacro:property name="caster_wheel_offset_z" value="${-wheel_offset_z - wheel_radius + caster_wheel_radius}"/>
     <material name="white">
         <color rgba="1 1 1 1" />

Commit message: Update caster wheel X offset calculation
Changed the caster_wheel_offset_x property to be calculated as chassis_length minus 0.03 instead of a fixed value. This makes the caster wheel position relative to the chassis length, improving model flexibility.

File: description/robot_core.xacro (robot description, xacro)
@@ -14,5 +14,5 @@
     <xacro:property name="caster_wheel_radius" value="0.01"/>
     <xacro:property name="caster_wheel_mass" value="0.01"/>
-    <xacro:property name="caster_wheel_offset_x" value="0.03"/>
+    <xacro:property name="caster_wheel_offset_x" value="${chassis_length - 0.03}"/>
     <xacro:property name="caster_wheel_offset_z" value="${-wheel_offset_z - wheel_radius + caster_wheel_radius}"/>
     <material name="white">
